Commit message: Change ur_description package name to moveit_resources_ur_description

File: ur_description/urdf/ur.urdf.xacro (robot description, xacro)
@@ -4,5 +4,5 @@
    <xacro:arg name="name" default="ur"/>
    <!-- import main macro -->
-   <xacro:include filename="$(find ur_description)/urdf/ur_macro.xacro"/>
+   <xacro:include filename="$(find moveit_resources_ur_description)/urdf/ur_macro.xacro"/>
    <!-- possible 'ur_type' values: ur3, ur3e, ur5, ur5e, ur10, ur10e, ur16e, ur20 -->
    <!-- the default value should raise an error in case this was called without defining the type -->
@@ -10,8 +10,8 @@
    <!-- parameters -->
    <xacro:arg name="tf_prefix" default="" />
-   <xacro:arg name="joint_limit_params" default="$(find ur_description)/config/$(arg ur_type)/joint_limits.yaml"/>
-   <xacro:arg name="kinematics_params" default="$(find ur_description)/config/$(arg ur_type)/default_kinematics.yaml"/>
-   <xacro:arg name="physical_params" default="$(find ur_description)/config/$(arg ur_type)/physical_parameters.yaml"/>
-   <xacro:arg name="visual_params" default="$(find ur_description)/config/$(arg ur_type)/visual_parameters.yaml"/>
+   <xacro:arg name="joint_limit_params" default="$(find moveit_resources_ur_description)/config/$(arg ur_type)/joint_limits.yaml"/>
+   <xacro:arg name="kinematics_params" default="$(find moveit_resources_ur_description)/config/$(arg ur_type)/default_kinematics.yaml"/>
+   <xacro:arg name="physical_params" default="$(find moveit_resources_ur_description)/config/$(arg ur_type)/physical_parameters.yaml"/>
+   <xacro:arg name="visual_params" default="$(find moveit_resources_ur_description)/config/$(arg ur_type)/visual_parameters.yaml"/>
    <xacro:arg name="transmission_hw_interface" default=""/>
    <xacro:arg name="safety_limits" default="false"/>
@@ -46,5 +46,5 @@
    <xacro:arg name="simulation_controllers" default="" />
    <!-- initial position for simulations (Fake Hardware, Gazebo, Ignition) -->
-   <xacro:arg name="initial_positions_file" default="$(find ur_description)/config/initial_positions.yaml"/>
+   <xacro:arg name="initial_positions_file" default="$(find moveit_resources_ur_description)/config/initial_positions.yaml"/>
    <!-- convert to property to use substitution in function -->
    <xacro:property name="initial_positions_file" default="$(arg initial_positions_file)"/>
@@ -56,5 +56,5 @@
       xyz="0 0 0" rpy="0 0 0" />
      <geometry>
-      <mesh filename="package://ur_description/meshes/ur3/bench_simplified_corrected.stl" />
+      <mesh filename="package://moveit_resources_ur_description/meshes/ur3/bench_simplified_corrected.stl" />
      </geometry>
      <material name="">
@@ -66,5 +66,5 @@
       xyz="0 0 0" rpy="0 0 0" />
      <geometry>
-      <mesh filename="package://ur_description/meshes/ur3/bench_simplified_corrected.stl" />
+      <mesh filename="package://moveit_resources_ur_description/meshes/ur3/bench_simplified_corrected.stl" />
      </geometry>
     </collision>

File: ur_description/urdf/ur_macro.xacro (robot description, xacro)
@@ -42,6 +42,6 @@
      - Muhammad Asif Rana
   -->
-  <xacro:include filename="$(find ur_description)/urdf/inc/ur_transmissions.xacro" />
-  <xacro:include filename="$(find ur_description)/urdf/inc/ur_common.xacro" />
+  <xacro:include filename="$(find moveit_resources_ur_description)/urdf/inc/ur_transmissions.xacro" />
+  <xacro:include filename="$(find moveit_resources_ur_description)/urdf/inc/ur_common.xacro" />
   <xacro:macro name="ur_robot" params="
     name
@@ -94,5 +94,5 @@
     <xacro:if value="${generate_ros2_control_tag}">
       <!-- ros2 control include -->
-      <xacro:include filename="$(find ur_description)/urdf/ur.ros2_control.xacro" />
+      <xacro:include filename="$(find moveit_resources_ur_description)/urdf/ur.ros2_control.xacro" />
       <!-- ros2 control instance -->
       <xacro:ur_ros2_control

Commit message: Revert package name back to ur_description

File: ur_description/urdf/ur.urdf.xacro (robot description, xacro)
@@ -4,5 +4,5 @@
    <xacro:arg name="name" default="ur"/>
    <!-- import main macro -->
-   <xacro:include filename="$(find moveit_resources_ur_description)/urdf/ur_macro.xacro"/>
+   <xacro:include filename="$(find ur_description)/urdf/ur_macro.xacro"/>
    <!-- possible 'ur_type' values: ur3, ur3e, ur5, ur5e, ur10, ur10e, ur16e, ur20 -->
    <!-- the default value should raise an error in case this was called without defining the type -->
@@ -10,8 +10,8 @@
    <!-- parameters -->
    <xacro:arg name="tf_prefix" default="" />
-   <xacro:arg name="joint_limit_params" default="$(find moveit_resources_ur_description)/config/$(arg ur_type)/joint_limits.yaml"/>
-   <xacro:arg name="kinematics_params" default="$(find moveit_resources_ur_description)/config/$(arg ur_type)/default_kinematics.yaml"/>
-   <xacro:arg name="physical_params" default="$(find moveit_resources_ur_description)/config/$(arg ur_type)/physical_parameters.yaml"/>
-   <xacro:arg name="visual_params" default="$(find moveit_resources_ur_description)/config/$(arg ur_type)/visual_parameters.yaml"/>
+   <xacro:arg name="joint_limit_params" default="$(find ur_description)/config/$(arg ur_type)/joint_limits.yaml"/>
+   <xacro:arg name="kinematics_params" default="$(find ur_description)/config/$(arg ur_type)/default_kinematics.yaml"/>
+   <xacro:arg name="physical_params" default="$(find ur_description)/config/$(arg ur_type)/physical_parameters.yaml"/>
+   <xacro:arg name="visual_params" default="$(find ur_description)/config/$(arg ur_type)/visual_parameters.yaml"/>
    <xacro:arg name="transmission_hw_interface" default=""/>
    <xacro:arg name="safety_limits" default="false"/>
@@ -46,5 +46,5 @@
    <xacro:arg name="simulation_controllers" default="" />
    <!-- initial position for simulations (Fake Hardware, Gazebo, Ignition) -->
-   <xacro:arg name="initial_positions_file" default="$(find moveit_resources_ur_description)/config/initial_positions.yaml"/>
+   <xacro:arg name="initial_positions_file" default="$(find ur_description)/config/initial_positions.yaml"/>
    <!-- convert to property to use substitution in function -->
    <xacro:property name="initial_positions_file" default="$(arg initial_positions_file)"/>
@@ -56,5 +56,5 @@
       xyz="0 0 0" rpy="0 0 0" />
      <geometry>
-      <mesh filename="package://moveit_resources_ur_description/meshes/ur3/bench_simplified_corrected.stl" />
+      <mesh filename="package://ur_description/meshes/ur3/bench_simplified_corrected.stl" />
      </geometry>
      <material name="">
@@ -66,5 +66,5 @@
       xyz="0 0 0" rpy="0 0 0" />
      <geometry>
-      <mesh filename="package://moveit_resources_ur_description/meshes/ur3/bench_simplified_corrected.stl" />
+      <mesh filename="package://ur_description/meshes/ur3/bench_simplified_corrected.stl" />
      </geometry>
     </collision>

File: ur_description/urdf/ur_macro.xacro (robot description, xacro)
@@ -42,6 +42,6 @@
      - Muhammad Asif Rana
   -->
-  <xacro:include filename="$(find moveit_resources_ur_description)/urdf/inc/ur_transmissions.xacro" />
-  <xacro:include filename="$(find moveit_resources_ur_description)/urdf/inc/ur_common.xacro" />
+  <xacro:include filename="$(find ur_description)/urdf/inc/ur_transmissions.xacro" />
+  <xacro:include filename="$(find ur_description)/urdf/inc/ur_common.xacro" />
   <xacro:macro name="ur_robot" params="
     name
@@ -94,5 +94,5 @@
     <xacro:if value="${generate_ros2_control_tag}">
       <!-- ros2 control include -->
-      <xacro:include filename="$(find moveit_resources_ur_description)/urdf/ur.ros2_control.xacro" />
+      <xacro:include filename="$(find ur_description)/urdf/ur.ros2_control.xacro" />
       <!-- ros2 control instance -->
       <xacro:ur_ros2_control
