Commit message: Add second robot to workspace

File: crm_dual_robot_cell/crm_dual_description/urdf/crm_dual.urdf.xacro (robot description, xacro)
@@ -1,31 +1,93 @@
 <?xml version="1.0"?>
-<robot name="my_dual_robot_cell" xmlns:xacro="http://ros.org/wiki/xacro">
-  <xacro:include filename="$(find crm_description)/urdf/crm_dual_macro.xacro"/>
-  <xacro:arg name="alice_ur_type" default="ur3"/>
-  <xacro:arg name="alice_joint_limits_parameters_file" default="$(find ur_description)/config/$(arg alice_ur_type)/joint_limits.yaml"/>
-  <xacro:arg name="alice_kinematics_parameters_file" default="$(find ur_description)/config/$(arg alice_ur_type)/default_kinematics.yaml"/>
-  <xacro:arg name="alice_physical_parameters_file" default="$(find ur_description)/config/$(arg alice_ur_type)/physical_parameters.yaml"/>
-  <xacro:arg name="alice_visual_parameters_file" default="$(find ur_description)/config/$(arg alice_ur_type)/visual_parameters.yaml"/>
-  <xacro:arg name="bob_ur_type" default="ur3"/>
-  <xacro:arg name="bob_joint_limits_parameters_file" default="$(find ur_description)/config/$(arg bob_ur_type)/joint_limits.yaml"/>
-  <xacro:arg name="bob_kinematics_parameters_file" default="$(find ur_description)/config/$(arg bob_ur_type)/default_kinematics.yaml"/>
-  <xacro:arg name="bob_physical_parameters_file" default="$(find ur_description)/config/$(arg bob_ur_type)/physical_parameters.yaml"/>
-  <xacro:arg name="bob_visual_parameters_file" default="$(find ur_description)/config/$(arg bob_ur_type)/visual_parameters.yaml"/>
-  <link name="world"/>
-  <!--This will create the scene where the robot is located in-->
-  <xacro:my_dual_robot_cell
-    parent="world"
-    alice_ur_type="$(arg alice_ur_type)"
-    alice_joint_limits_parameters_file="$(arg alice_joint_limits_parameters_file)"
-    alice_kinematics_parameters_file="$(arg alice_kinematics_parameters_file)"
-    alice_physical_parameters_file="$(arg alice_physical_parameters_file)"
-    alice_visual_parameters_file="$(arg alice_visual_parameters_file)"
-    bob_ur_type="$(arg bob_ur_type)"
-    bob_joint_limits_parameters_file="$(arg bob_joint_limits_parameters_file)"
-    bob_kinematics_parameters_file="$(arg bob_kinematics_parameters_file)"
-    bob_physical_parameters_file="$(arg bob_physical_parameters_file)"
-    bob_visual_parameters_file="$(arg bob_visual_parameters_file)"
-    >
-      <origin xyz="0 0 0.78" rpy="0 0 0" />
-  </xacro:my_dual_robot_cell>
+<robot xmlns:xacro="http://wiki.ros.org/xacro" name="crm_robot">
+   <!-- robot name parameter -->
+   <xacro:arg name="name" default="right_ur3"/>
+   <!-- import main macro -->
+   <xacro:include filename="$(find crm_dual_description)/urdf/crm_dual_macro.xacro"/>
+   <!-- possible 'ur_type' values: ur3, ur3e, ur5, ur5e, ur10, ur10e, ur16e, ur20 -->
+   <!-- the default value should raise an error in case this was called without defining the type -->
+   <xacro:arg name="ur_type" default="ur3"/>
+   <!-- parameters -->
+   <xacro:arg name="tf_prefix" default="" />
+   <xacro:arg name="joint_limit_params" default="$(find ur_description)/config/$(arg ur_type)/joint_limits.yaml"/>
+   <xacro:arg name="kinematics_params" default="$(find ur_description)/config/$(arg ur_type)/default_kinematics.yaml"/>
+   <xacro:arg name="physical_params" default="$(find ur_description)/config/$(arg ur_type)/physical_parameters.yaml"/>
+   <xacro:arg name="visual_params" default="$(find ur_description)/config/$(arg ur_type)/visual_parameters.yaml"/>
+   <xacro:arg name="transmission_hw_interface" default=""/>
+   <xacro:arg name="safety_limits" default="false"/>
+   <xacro:arg name="safety_pos_margin" default="0.15"/>
+   <xacro:arg name="safety_k_position" default="20"/>
+   <!-- ros2_control related parameters -->
+   <xacro:arg name="headless_mode" default="false" />
+   <xacro:arg name="robot_ip" default="0.0.0.0" />
+   <xacro:arg name="script_filename" default=""/>
+   <xacro:arg name="output_recipe_filename" default=""/>
+   <xacro:arg name="input_recipe_filename" default=""/>
+   <xacro:arg name="reverse_ip" default="0.0.0.0"/>
+   <xacro:arg name="script_command_port" default="50004"/>
+   <xacro:arg name="reverse_port" default="50001"/>
+   <xacro:arg name="script_sender_port" default="50002"/>
+   <xacro:arg name="trajectory_port" default="50003"/>
+   <!--   tool communication related parameters-->
+   <xacro:arg name="use_tool_communication" default="false" />
+   <xacro:arg name="tool_voltage" default="0" />
+   <xacro:arg name="tool_parity" default="0" />
+   <xacro:arg name="tool_baud_rate" default="115200" />
+   <xacro:arg name="tool_stop_bits" default="1" />
+   <xacro:arg name="tool_rx_idle_chars" default="1.5" />
+   <xacro:arg name="tool_tx_idle_chars" default="3.5" />
+   <xacro:arg name="tool_device_name" default="/tmp/ttyUR" />
+   <xacro:arg name="tool_tcp_port" default="54321" />
+   <!-- Simulation parameters -->
+   <xacro:arg name="use_fake_hardware" default="false" />
+   <xacro:arg name="fake_sensor_commands" default="false" />
+   <xacro:arg name="sim_gazebo" default="false" />
+   <xacro:arg name="sim_ignition" default="false" />
+   <xacro:arg name="simulation_controllers" default="" />
+   <!-- initial position for simulations (Fake Hardware, Gazebo, Ignition) -->
+   <xacro:arg name="initial_positions_file" default="$(find crm_description)/config/initial_positions.yaml"/>
+   <!-- convert to property to use substitution in function -->
+   <xacro:property name="initial_positions_file" default="$(arg initial_positions_file)"/>
+   <!-- create link fixed to the "world" -->
+   <link name="world" />
+   <!-- right arm -->
+   <xacro:crm_robot
+     name=""
+     tf_prefix=""
+     parent="world"
+     joint_limits_parameters_file="$(arg joint_limit_params)"
+     kinematics_parameters_file="$(arg kinematics_params)"
+     physical_parameters_file="$(arg physical_params)"
+     visual_parameters_file="$(arg visual_params)"
+     transmission_hw_interface="$(arg transmission_hw_interface)"
+     safety_limits="$(arg safety_limits)"
+     safety_pos_margin="$(arg safety_pos_margin)"
+     safety_k_position="$(arg safety_k_position)"
+     use_fake_hardware="$(arg use_fake_hardware)"
+     fake_sensor_commands="$(arg fake_sensor_commands)"
+     sim_gazebo="$(arg sim_gazebo)"
+     sim_ignition="$(arg sim_ignition)"
+     headless_mode="$(arg headless_mode)"
+     initial_positions="${xacro.load_yaml(initial_positions_file)}"
+     use_tool_communication="$(arg use_tool_communication)"
+     tool_voltage="$(arg tool_voltage)"
+     tool_parity="$(arg tool_parity)"
+     tool_baud_rate="$(arg tool_baud_rate)"
+     tool_stop_bits="$(arg tool_stop_bits)"
+     tool_rx_idle_chars="$(arg tool_rx_idle_chars)"
+     tool_tx_idle_chars="$(arg tool_tx_idle_chars)"
+     tool_device_name="$(arg tool_device_name)"
+     tool_tcp_port="$(arg tool_tcp_port)"
+     robot_ip="$(arg robot_ip)"
+     script_filename="$(arg script_filename)"
+     output_recipe_filename="$(arg output_recipe_filename)"
+     input_recipe_filename="$(arg input_recipe_filename)"
+     reverse_ip="$(arg reverse_ip)"
+     script_command_port="$(arg script_command_port)"
+     reverse_port="$(arg reverse_port)"
+     script_sender_port="$(arg script_sender_port)"
+     trajectory_port="$(arg trajectory_port)"
+     >
+     <origin xyz="0 0 0.776572" rpy="0 0 0" />
+   </xacro:crm_robot>
 </robot>

File: crm_dual_robot_cell/crm_dual_description/urdf/crm_dual_macro.xacro (robot description, xacro)
@@ -2,18 +2,46 @@
 <robot xmlns:xacro="http://wiki.ros.org/xacro">
   <xacro:include filename="$(find ur_description)/urdf/ur_macro.xacro"/>
-  <xacro:macro name="my_dual_robot_cell" params="
+  <xacro:macro name="crm_robot" params="
+    name
+    tf_prefix
     parent
     *origin
-    alice_ur_type
-    bob_ur_type
-    alice_joint_limits_parameters_file
-    bob_joint_limits_parameters_file
-    alice_kinematics_parameters_file
-    bob_kinematics_parameters_file
-    alice_physical_parameters_file
-    bob_physical_parameters_file
-    alice_visual_parameters_file
-    bob_visual_parameters_file
-    ">
+    joint_limits_parameters_file
+    kinematics_parameters_file
+    physical_parameters_file
+    visual_parameters_file
+    generate_ros2_control_tag:=true
+    transmission_hw_interface:=hardware_interface/PositionJointInterface
+    safety_limits:=false
+    safety_pos_margin:=0.15
+    safety_k_position:=20
+    use_fake_hardware:=false
+    fake_sensor_commands:=false
+    sim_gazebo:=false
+    sim_ignition:=false
+    headless_mode:=false
+    initial_positions:=${dict(shoulder_pan_joint=0.0,shoulder_lift_joint=-1.57,elbow_joint=0.0,wrist_1_joint=-1.57,wrist_2_joint=0.0,wrist_3_joint=0.0)}
+    use_tool_communication:=false
+    tool_voltage:=0
+    tool_parity:=0
+    tool_baud_rate:=115200
+    tool_stop_bits:=1
+    tool_rx_idle_chars:=1.5
+    tool_tx_idle_chars:=3.5
+    tool_device_name:=/tmp/ttyUR
+    tool_tcp_port:=54321
+    robot_ip:=0.0.0.0
+    script_filename:=to_be_filled_by_ur_robot_driver
+    output_recipe_filename:=to_be_filled_by_ur_robot_driver
+    input_recipe_filename:=to_be_filled_by_ur_robot_driver
+    reverse_port:=50001
+    script_sender_port:=50002
+    reverse_ip:=0.0.0.0
+    script_command_port:=50004
+    trajectory_port:=50003
+    non_blocking_read:=true
+    keep_alive_count:=2"
+    >
+    <!-- Base and mount setup -->
     <joint name="vention_bench_base_joint" type="fixed">
       <xacro:insert_block name="origin" />
@@ -26,5 +54,8 @@
           <mesh filename="package://crm_description/meshes/bench_simplified_corrected.stl"/>
         </geometry>
-        <origin rpy="0 0 ${pi}" xyz="0 0.73 -0.78"/>
+        <origin rpy="0 0 ${pi}" xyz="0 0.72 -0.776572"/>
+        <material name="custom_blue">
+          <color rgba="${106/255} ${165/255} ${219/255} 1.0"/>
+        </material>
       </visual>
       <collision>
@@ -32,43 +63,99 @@
           <mesh filename="package://crm_description/meshes/bench_simplified_corrected.stl"/>
         </geometry>
-        <origin rpy="0 0 ${pi}" xyz="0 0.73 -0.78"/>
+        <origin rpy="0 0 ${pi}" xyz="0 0.72 -0.776572"/>
       </collision>
     </link>
-    <link name="bob_robot_mount"/>
-    <joint name="base_to_bob_robot_mount" type="fixed">
+    <link name="right_ur3_robot_mount"/>
+    <joint name="right_ur3_base_to_robot_mount" type="fixed">
       <parent link="vention_bench"/>
-      <child link="bob_robot_mount"/>
-      <origin xyz="0.315 0.6 0.01" rpy="0 0 ${pi}" />
+      <child link="right_ur3_robot_mount"/>
+      <origin xyz="0.315 0.607 0.0145" rpy="0 0 ${pi}" />
     </joint>
-    <link name="alice_robot_mount"/>
-    <joint name="base_to_alice_robot_mount" type="fixed">
+    <link name="left_ur3_robot_mount"/>
+    <joint name="left_ur3_base_to_robot_mount" type="fixed">
       <parent link="vention_bench"/>
-      <child link="alice_robot_mount"/>
-      <origin xyz="-0.315 0.6 0.01" rpy="0 0 ${pi}" />
+      <child link="left_ur3_robot_mount"/>
+      <origin xyz="-0.315 0.607 0.0145" rpy="0 0 ${pi}" />
     </joint>
-    <!--This will create the first robot-->
+    <!-- Right arm -->
     <xacro:ur_robot
-      name="alice"
-      tf_prefix="alice_"
-      parent="alice_robot_mount"
-      joint_limits_parameters_file="${alice_joint_limits_parameters_file}"
-      kinematics_parameters_file="${alice_kinematics_parameters_file}"
-      physical_parameters_file="${alice_physical_parameters_file}"
-      visual_parameters_file="${alice_visual_parameters_file}"
-    >
-      <origin xyz="0 0 0" rpy="0 0 0" />
-    </xacro:ur_robot>
-    <!--This will create the second robot-->
+     name="right_ur3"
+     tf_prefix="right_ur3_"
+     parent="right_ur3_robot_mount"
+     joint_limits_parameters_file="$(arg joint_limit_params)"
+     kinematics_parameters_file="$(arg kinematics_params)"
+     physical_parameters_file="$(arg physical_params)"
+     visual_parameters_file="$(arg visual_params)"
+     transmission_hw_interface="$(arg transmission_hw_interface)"
+     safety_limits="$(arg safety_limits)"
+     safety_pos_margin="$(arg safety_pos_margin)"
+     safety_k_position="$(arg safety_k_position)"
+     use_fake_hardware="$(arg use_fake_hardware)"
+     fake_sensor_commands="$(arg fake_sensor_commands)"
+     sim_gazebo="$(arg sim_gazebo)"
+     sim_ignition="$(arg sim_ignition)"
+     headless_mode="$(arg headless_mode)"
+     initial_positions="${xacro.load_yaml(initial_positions_file)}"
+     use_tool_communication="$(arg use_tool_communication)"
+     tool_voltage="$(arg tool_voltage)"
+     tool_parity="$(arg tool_parity)"
+     tool_baud_rate="$(arg tool_baud_rate)"
+     tool_stop_bits="$(arg tool_stop_bits)"
+     tool_rx_idle_chars="$(arg tool_rx_idle_chars)"
+     tool_tx_idle_chars="$(arg tool_tx_idle_chars)"
+     tool_device_name="$(arg tool_device_name)"
+     tool_tcp_port="$(arg tool_tcp_port)"
+     robot_ip="$(arg robot_ip)"
+     script_filename="$(arg script_filename)"
+     output_recipe_filename="$(arg output_recipe_filename)"
+     input_recipe_filename="$(arg input_recipe_filename)"
+     reverse_ip="$(arg reverse_ip)"
+     script_command_port="$(arg script_command_port)"
+     reverse_port="$(arg reverse_port)"
+     script_sender_port="$(arg script_sender_port)"
+     trajectory_port="$(arg trajectory_port)"
+     >
+     <origin xyz="0 0 0" rpy="0 0 0" />
+   </xacro:ur_robot>
+    <!-- Left arm, identical to the right arm but with a different tf_prefix -->
     <xacro:ur_robot
-      name="bob"
-      tf_prefix="bob_"
-      parent="bob_robot_mount"
-      joint_limits_parameters_file="${bob_joint_limits_parameters_file}"
-      kinematics_parameters_file="${bob_kinematics_parameters_file}"
-      physical_parameters_file="${bob_physical_parameters_file}"
-      visual_parameters_file="${bob_visual_parameters_file}"
-    >
-      <origin xyz="0 0 0" rpy="0 0 0" />
-    </xacro:ur_robot>
+     name="left_ur3"
+     tf_prefix="left_ur3_"
+     parent="left_ur3_robot_mount"
+     joint_limits_parameters_file="$(arg joint_limit_params)"
+     kinematics_parameters_file="$(arg kinematics_params)"
+     physical_parameters_file="$(arg physical_params)"
+     visual_parameters_file="$(arg visual_params)"
+     transmission_hw_interface="$(arg transmission_hw_interface)"
+     safety_limits="$(arg safety_limits)"
+     safety_pos_margin="$(arg safety_pos_margin)"
+     safety_k_position="$(arg safety_k_position)"
+     use_fake_hardware="$(arg use_fake_hardware)"
+     fake_sensor_commands="$(arg fake_sensor_commands)"
+     sim_gazebo="$(arg sim_gazebo)"
+     sim_ignition="$(arg sim_ignition)"
+     headless_mode="$(arg headless_mode)"
+     initial_positions="${xacro.load_yaml(initial_positions_file)}"
+     use_tool_communication="$(arg use_tool_communication)"
+     tool_voltage="$(arg tool_voltage)"
+     tool_parity="$(arg tool_parity)"
+     tool_baud_rate="$(arg tool_baud_rate)"
+     tool_stop_bits="$(arg tool_stop_bits)"
+     tool_rx_idle_chars="$(arg tool_rx_idle_chars)"
+     tool_tx_idle_chars="$(arg tool_tx_idle_chars)"
+     tool_device_name="$(arg tool_device_name)"
+     tool_tcp_port="$(arg tool_tcp_port)"
+     robot_ip="$(arg robot_ip)"
+     script_filename="$(arg script_filename)"
+     output_recipe_filename="$(arg output_recipe_filename)"
+     input_recipe_filename="$(arg input_recipe_filename)"
+     reverse_ip="$(arg reverse_ip)"
+     script_command_port="$(arg script_command_port)"
+     reverse_port="$(arg reverse_port)"
+     script_sender_port="$(arg script_sender_port)"
+     trajectory_port="$(arg trajectory_port)"
+     >
+     <origin xyz="0 0 0" rpy="0 0 0" />
+   </xacro:ur_robot>
   </xacro:macro>
 </robot>
