Commit message: Fix alice and bob robot positions

File: crm_dual_robot_cell/crm_dual_description/urdf/crm_dual_macro.xacro (robot description, xacro)
@@ -28,5 +28,5 @@
         <origin rpy="0 0 ${pi}" xyz="0 0.72 -0.776572"/>
         <material name="custom_blue">
-          <color rgba="${106/255} ${165/255} ${219/255} 1.0"/>
+          <color rgba="0.4157 0.6471 0.8588 1.0"/>
         </material>
       </visual>
@@ -43,5 +43,5 @@
       <parent link="vention_bench"/>
       <child link="alice_robot_mount"/>
-      <origin xyz="0.315 0.607 0.0145" rpy="0 0 ${pi}" />
+      <origin xyz="-0.315 0.607 0.0145" rpy="0 0 ${pi}" />
     </joint>
     <link name="bob_robot_mount"/>
@@ -49,5 +49,5 @@
       <parent link="vention_bench"/>
       <child link="bob_robot_mount"/>
-      <origin xyz="-0.315 0.607 0.0145" rpy="0 0 ${pi}" />
+      <origin xyz="0.315 0.607 0.0145" rpy="0 0 ${pi}" />
     </joint>
     <!--Creates the 1st Robot-->

Commit message: Update urdf

File: crm_dual_robot_cell/crm_dual_description/urdf/crm_dual_macro.xacro (robot description, xacro)
@@ -2,4 +2,7 @@
 <robot xmlns:xacro="http://ros.org/wiki/xacro">
   <xacro:include filename="$(find ur_description)/urdf/ur_macro.xacro"/>
+  <material name="blue">
+    <color rgba="0 0 0.8 1"/>
+  </material>
   <xacro:macro name="crm_dual_robot" params="
     parent
@@ -75,4 +78,56 @@
       <origin xyz="0 0 0" rpy="0 0 0" />
     </xacro:ur_robot>
+    <link name="bob_bltouch"/>
+    <joint name="bob_wrist_3-bltouch" type="fixed">
+      <parent link="bob_wrist_3_link" />
+      <child link="bob_bltouch" />
+      <origin xyz="0.0674 0 0.0206502" rpy="0 ${pi/2} ${pi}" />
+    </joint>
+    <link name="bob_hotend">
+        <visual>
+          <geometry>
+            <mesh filename="package://crm_dual_description/meshes/end_effector_updated_bltouch.stl"/>
+          </geometry>
+          <origin rpy="0 0 0" xyz="0 0 0"/>
+          <material name="blue"/>
+        </visual>
+        <collision>
+          <geometry>
+            <mesh filename="package://crm_dual_description/meshes/end_effector_updated_bltouch.stl"/>
+          </geometry>
+          <origin rpy="0 0 0" xyz="0 0 0"/>
+        </collision>
+    </link>
+    <joint name="bob_tool0-hotend" type="fixed">
+      <parent link="bob_tool0"/>
+      <child link="bob_hotend"/>
+      <origin xyz="0 0 0" rpy="0 ${pi/2} ${pi}" />
+    </joint>
+    <link name="bob_nozzle"/>
+    <joint name="bob_tool0-nozzle" type="fixed">
+      <parent link="bob_tool0" />
+      <child link="bob_nozzle" />
+      <origin xyz="0.002 0.05 0.1368" rpy="${pi} 0 0" />
+    </joint>
+    <link name="alice_laser_profiler">
+        <visual>
+          <geometry>
+            <mesh filename="package://crm_dual_description/meshes/laser_profiler.stl"/>
+          </geometry>
+          <origin rpy="0 0 0" xyz="0 0 0"/>
+          <material name="blue"/>
+        </visual>
+        <collision>
+          <geometry>
+            <mesh filename="package://crm_dual_description/meshes/laser_profiler.stl"/>
+          </geometry>
+          <origin rpy="0 0 0" xyz="0 0 0"/>
+        </collision>
+    </link>
+    <joint name="alice_tool0-laser_profiler" type="fixed">
+      <parent link="alice_tool0"/>
+      <child link="alice_laser_profiler"/>
+      <origin xyz="0 0 0" rpy="0 ${pi} 0" />
+    </joint>
   </xacro:macro>
 </robot>

Commit message: Update bob urdf

File: crm_dual_robot_cell/crm_dual_description/urdf/crm_dual_macro.xacro (robot description, xacro)
@@ -78,10 +78,4 @@
       <origin xyz="0 0 0" rpy="0 0 0" />
     </xacro:ur_robot>
-    <link name="bob_bltouch"/>
-    <joint name="bob_wrist_3-bltouch" type="fixed">
-      <parent link="bob_wrist_3_link" />
-      <child link="bob_bltouch" />
-      <origin xyz="0.0674 0 0.0206502" rpy="0 ${pi/2} ${pi}" />
-    </joint>
     <link name="bob_hotend">
         <visual>
@@ -89,5 +83,5 @@
             <mesh filename="package://crm_dual_description/meshes/end_effector_updated_bltouch.stl"/>
           </geometry>
-          <origin rpy="0 0 0" xyz="0 0 0"/>
+          <origin rpy="${-pi/2} 0 ${-pi/2}" xyz="0.003186 0.021844 0"/>
           <material name="blue"/>
         </visual>
@@ -102,5 +96,5 @@
       <parent link="bob_tool0"/>
       <child link="bob_hotend"/>
-      <origin xyz="0 0 0" rpy="0 ${pi/2} ${pi}" />
+      <origin xyz="0 0 0" rpy="0 0 0" />
     </joint>
     <link name="bob_nozzle"/>
@@ -110,4 +104,16 @@
       <origin xyz="0.002 0.05 0.1368" rpy="${pi} 0 0" />
     </joint>
+    <link name="bob_bltouch"/>
+    <joint name="bob_tool0-bltouch" type="fixed">
+      <parent link="bob_tool0" />
+      <child link="bob_bltouch" />
+      <origin xyz="-0.024252 0.026407 0.156326" rpy="${pi} 0 0" />
+    </joint>
+    <!-- Old BLTouch Config -->
+    <!-- <joint name="bob_tool0-bltouch" type="fixed">
+      <parent link="bob_tool0" />
+      <child link="bob_bltouch" />
+      <origin xyz="0.0674 0 0.0206502" rpy="0 ${pi/2} ${pi}" />
+    </joint> -->
     <link name="alice_laser_profiler">
         <visual>

File: crm_single_robot_cell/crm_description/urdf/ur_macro.xacro (robot description, xacro)
@@ -304,5 +304,5 @@
     <!-- ROS-Industrial 'tool0' frame - all-zeros tool frame -->
     <link name="${tf_prefix}tool0">
-        <visual>
+        <!-- <visual>
           <geometry>
             <mesh filename="package://crm_description/meshes/end_effector_thermal_camera.stl"/>
@@ -318,9 +318,9 @@
           </geometry>
           <origin rpy="${-pi/2} 0 ${-pi/2}" xyz="0.003186 0.021844 0"/>
-        </collision>
+        </collision> -->
     </link>
     <joint name="${tf_prefix}flange-tool0" type="fixed">
       <!-- default toolframe - X+ left, Y+ up, Z+ front -->
-      <origin xyz="0 0 0" rpy="${pi/2.0} 0 ${pi/2.0}"/>
+      <origin xyz="0 0 0" rpy="0 0 0"/>
       <parent link="${tf_prefix}flange"/>
       <child link="${tf_prefix}tool0"/>

Commit message: Update color and add collision pose for hotend link

File: crm_dual_robot_cell/crm_dual_description/urdf/crm_dual_macro.xacro (robot description, xacro)
@@ -2,6 +2,6 @@
 <robot xmlns:xacro="http://ros.org/wiki/xacro">
   <xacro:include filename="$(find ur_description)/urdf/ur_macro.xacro"/>
-  <material name="blue">
-    <color rgba="0 0 0.8 1"/>
+  <material name="custom_gray">
+    <color rgba="0.24705882352941178 0.34509803921568627 0.40784313725490196 1"/>
   </material>
   <xacro:macro name="crm_dual_robot" params="
@@ -84,5 +84,5 @@
           </geometry>
           <origin rpy="${-pi/2} 0 ${-pi/2}" xyz="0.003186 0.021844 0"/>
-          <material name="blue"/>
+          <material name="custom_gray"/>
         </visual>
         <collision>
@@ -90,5 +90,5 @@
             <mesh filename="package://crm_dual_description/meshes/end_effector_updated_bltouch.stl"/>
           </geometry>
-          <origin rpy="0 0 0" xyz="0 0 0"/>
+          <origin rpy="${-pi/2} 0 ${-pi/2}" xyz="0.003186 0.021844 0"/>
         </collision>
     </link>
@@ -122,5 +122,5 @@
           </geometry>
           <origin rpy="0 0 0" xyz="0 0 0"/>
-          <material name="blue"/>
+          <material name="custom_gray"/>
         </visual>
         <collision>

Commit message: Approximate laser profiler position

File: crm_dual_robot_cell/crm_dual_description/urdf/crm_dual_macro.xacro (robot description, xacro)
@@ -121,5 +121,5 @@
             <mesh filename="package://crm_dual_description/meshes/laser_profiler.stl"/>
           </geometry>
-          <origin rpy="0 0 0" xyz="0 0 0"/>
+          <origin rpy="0 0 0" xyz="-0.01 0.0075 0.0225"/>
           <material name="custom_gray"/>
         </visual>
@@ -128,5 +128,5 @@
             <mesh filename="package://crm_dual_description/meshes/laser_profiler.stl"/>
           </geometry>
-          <origin rpy="0 0 0" xyz="0 0 0"/>
+          <origin rpy="0 0 0" xyz="-0.01 0.0075 0.0225"/>
         </collision>
     </link>

Commit message: Fix vention table height

File: crm_dual_robot_cell/crm_dual_description/urdf/crm_dual_macro.xacro (robot description, xacro)
@@ -81,5 +81,5 @@
         <visual>
           <geometry>
-            <mesh filename="package://crm_dual_description/meshes/end_effector_updated_bltouch.stl"/>
+            <mesh filename="package://crm_dual_description/meshes/end_effector.stl"/>
           </geometry>
           <origin rpy="${-pi/2} 0 ${-pi/2}" xyz="0.003186 0.021844 0"/>
@@ -88,5 +88,5 @@
         <collision>
           <geometry>
-            <mesh filename="package://crm_dual_description/meshes/end_effector_updated_bltouch.stl"/>
+            <mesh filename="package://crm_dual_description/meshes/end_effector.stl"/>
           </geometry>
           <origin rpy="${-pi/2} 0 ${-pi/2}" xyz="0.003186 0.021844 0"/>

Commit message: Update end effector stl

File: crm_dual_robot_cell/crm_dual_description/urdf/crm_dual_macro.xacro (robot description, xacro)
@@ -81,5 +81,5 @@
         <visual>
           <geometry>
-            <mesh filename="package://crm_dual_description/meshes/end_effector.stl"/>
+            <mesh filename="package://crm_dual_description/meshes/end_effector_thermal_camera.stl"/>
           </geometry>
           <origin rpy="${-pi/2} 0 ${-pi/2}" xyz="0.003186 0.021844 0"/>
@@ -88,5 +88,5 @@
         <collision>
           <geometry>
-            <mesh filename="package://crm_dual_description/meshes/end_effector.stl"/>
+            <mesh filename="package://crm_dual_description/meshes/end_effector_thermal_camera.stl"/>
           </geometry>
           <origin rpy="${-pi/2} 0 ${-pi/2}" xyz="0.003186 0.021844 0"/>
