Commit message: Update bench height

File: crm_single_robot_cell/crm_description/urdf/crm.urdf.xacro (robot description, xacro)
@@ -89,5 +89,5 @@
      trajectory_port="$(arg trajectory_port)"
      >
-     <origin xyz="0 0 0.78" rpy="0 0 0" />
+     <origin xyz="0 0 0.776572" rpy="0 0 0" />
    </xacro:crm_robot>
    <xacro:if value="$(arg sim_gazebo)">

Commit message: Update urdf

File: crm_single_robot_cell/crm_description/urdf/crm.urdf.xacro (robot description, xacro)
@@ -2,5 +2,7 @@
 <robot name="crm_robot" xmlns:xacro="http://ros.org/wiki/xacro">
   <xacro:include filename="$(find crm_description)/urdf/crm_macro.xacro"/>
+  <xacro:arg name="name" default="right_ur3"/>
   <xacro:arg name="ur_type" default="ur3"/>
+  <xacro:arg name="tf_prefix" default="" />
   <xacro:arg name="joint_limits_parameters_file" default="$(find ur_description)/config/$(arg ur_type)/joint_limits.yaml"/>
   <xacro:arg name="kinematics_parameters_file" default="$(find ur_description)/config/$(arg ur_type)/default_kinematics.yaml"/>
@@ -10,6 +12,8 @@
   <!--This will create the scene where the robot is located in-->
   <xacro:crm_robot
+    name="right_ur3"
+    tf_prefix="right_ur3_"
     parent="world"
-    ur_type="$(arg ur_type)"
+    ur_type="ur3"
     joint_limits_parameters_file="$(arg joint_limits_parameters_file)"
     kinematics_parameters_file="$(arg kinematics_parameters_file)"
@@ -17,5 +21,5 @@
     visual_parameters_file="$(arg visual_parameters_file)"
     >
-      <origin xyz="0 0 0.78" rpy="0 0 0" />
+      <origin xyz="0 0 0.776572" rpy="0 0 0" />
   </xacro:crm_robot>
 </robot>

File: crm_single_robot_cell/crm_description/urdf/crm_macro.xacro (robot description, xacro)
@@ -1,10 +1,11 @@
 <?xml version="1.0"?>
 <robot xmlns:xacro="http://wiki.ros.org/xacro">
-  <xacro:include filename="$(find ur_description)/urdf/ur_macro.xacro" />
-  <xacro:macro name="crm_robot"
-    params="
+  <xacro:include filename="$(find crm_description)/urdf/ur_macro.xacro"/>
+  <xacro:macro name="crm_robot" params="
+    name
+    tf_prefix
     parent
+    ur_type
     *origin
-    ur_type
     joint_limits_parameters_file
     kinematics_parameters_file
@@ -20,25 +21,28 @@
       <visual>
         <geometry>
-          <mesh filename="package://crm_description/meshes/bench_simplified_corrected.stl" />
+          <mesh filename="package://crm_description/meshes/bench_simplified_corrected.stl"/>
         </geometry>
-        <origin rpy="0 0 ${pi}" xyz="0 0.73 -0.78" />
+        <origin rpy="0 0 ${pi}" xyz="0 0.72 -0.776572"/>
+        <material name="custom_blue">
+          <color rgba="${106/255} ${165/255} ${219/255} 1.0"/>
+        </material>
       </visual>
       <collision>
         <geometry>
-          <mesh filename="package://crm_description/meshes/bench_simplified_corrected.stl" />
+          <mesh filename="package://crm_description/meshes/bench_simplified_corrected.stl"/>
         </geometry>
-        <origin rpy="0 0 ${pi}" xyz="0 0.73 -0.78" />
+        <origin rpy="0 0 ${pi}" xyz="0 0.72 -0.776572"/>
       </collision>
     </link>
-    <link name="robot_mount" />
+    <link name="robot_mount"/>
     <joint name="base_to_robot_mount" type="fixed">
-      <parent link="vention_bench" />
-      <child link="robot_mount" />
-      <origin xyz="0.315 0.6 0.01" rpy="0 0 ${pi}" />
+      <parent link="vention_bench"/>
+      <child link="robot_mount"/>
+      <origin xyz="0.315 0.607 0.0145" rpy="0 0 ${pi}" />
     </joint>
     <!-- arm -->
     <xacro:ur_robot
-      name="${ur_type}"
-      tf_prefix="${ur_type}_"
+      name="right_ur3"
+      tf_prefix="right_ur3_"
       parent="robot_mount"
       joint_limits_parameters_file="${joint_limits_parameters_file}"
@@ -49,4 +53,10 @@
       <origin xyz="0 0 0" rpy="0 0 0" />
     </xacro:ur_robot>
+    <link name="right_ur3_bltouch"/>
+    <joint name="right_ur3_wrist_3-bltouch" type="fixed">
+      <parent link="right_ur3_wrist_3_link" />
+      <child link="right_ur3_bltouch" />
+      <origin xyz="0 0 0" rpy="${pi/2} 0 0" />
+    </joint>
   </xacro:macro>
 </robot>
