Commit message: Add bltouch link and update bench coordinates

File: crm_single_robot_cell/crm_description/urdf/crm_macro.xacro (robot description, xacro)
@@ -1,5 +1,5 @@
 <?xml version="1.0"?>
 <robot xmlns:xacro="http://wiki.ros.org/xacro">
-  <xacro:include filename="$(find ur_description)/urdf/ur_macro.xacro"/>
+  <xacro:include filename="$(find crm_description)/urdf/ur_macro.xacro"/>
   <xacro:macro name="crm_robot" params="
     name
@@ -53,5 +53,8 @@
           <mesh filename="package://crm_description/meshes/bench_simplified_corrected.stl"/>
         </geometry>
-        <origin rpy="0 0 ${pi}" xyz="0 0.73 -0.78"/>
+        <origin rpy="0 0 ${pi}" xyz="0 0.72 -0.776572"/>
+        <material name="custom_blue">
+          <color rgba="${106/255} ${165/255} ${219/255} 1.0"/>
+        </material>
       </visual>
       <collision>
@@ -59,5 +62,5 @@
           <mesh filename="package://crm_description/meshes/bench_simplified_corrected.stl"/>
         </geometry>
-        <origin rpy="0 0 ${pi}" xyz="0 0.73 -0.78"/>
+        <origin rpy="0 0 ${pi}" xyz="0 0.72 -0.776572"/>
       </collision>
     </link>
@@ -66,5 +69,5 @@
       <parent link="vention_bench"/>
       <child link="robot_mount"/>
-      <origin xyz="0.315 0.6 0.01" rpy="0 0 ${pi}" />
+      <origin xyz="0.315 0.607 0.0145" rpy="0 0 ${pi}" />
     </joint>
    <!-- arm -->
@@ -108,4 +111,10 @@
      <origin xyz="0 0 0" rpy="0 0 0" />
    </xacro:ur_robot>
+    <link name="right_ur3_bltouch"/>
+    <joint name="right_ur3_wrist_3-bltouch" type="fixed">
+      <parent link="right_ur3_wrist_3_link" />
+      <child link="right_ur3_bltouch" />
+      <origin xyz="0 0.0674 0.020661" rpy="0 ${pi/2} ${pi/2}" />
+    </joint>
   </xacro:macro>
 </robot>

Commit message: Clean Up

File: crm_single_robot_cell/crm_description/urdf/crm_macro.xacro (robot description, xacro)
@@ -115,5 +115,7 @@
       <parent link="right_ur3_wrist_3_link" />
       <child link="right_ur3_bltouch" />
-      <origin xyz="0 0.0674 0.020661" rpy="0 ${pi/2} ${pi/2}" />
+      <origin xyz="0 0 0" rpy="${pi/2} 0 0" />
+      <!-- <origin xyz="0 0 0" rpy="0 ${-pi/2} 0" /> -->
+      <!-- <origin xyz="0 0.0674 0.020661" rpy="0 ${pi/2} ${pi/2}" /> -->
     </joint>
   </xacro:macro>

Commit message: Set bltouch frame

File: crm_single_robot_cell/crm_description/urdf/crm_macro.xacro (robot description, xacro)
@@ -55,5 +55,5 @@
       <parent link="right_ur3_wrist_3_link" />
       <child link="right_ur3_bltouch" />
-      <origin xyz="0 0 0" rpy="${pi/2} 0 0" />
+      <origin xyz="0.0674 0 0.0206502" rpy="0 ${pi/2} ${pi}" />
     </joint>
   </xacro:macro>

Commit message: Add frame for nozzle (end effector)

File: crm_single_robot_cell/crm_description/urdf/crm_macro.xacro (robot description, xacro)
@@ -57,4 +57,10 @@
       <origin xyz="0.0674 0 0.0206502" rpy="0 ${pi/2} ${pi}" />
     </joint>
+    <link name="right_ur3_nozzle"/>
+    <joint name="right_ur3_wrist_3-nozzle" type="fixed">
+      <parent link="right_ur3_wrist_3_link" />
+      <child link="right_ur3_nozzle" />
+      <origin xyz="-0.002415 0.023405 0.1368" rpy="${pi} 0 0" />
+    </joint>
   </xacro:macro>
 </robot>

Commit message: Change nozzle parent link to tool0 and update nozzle position

File: crm_single_robot_cell/crm_description/urdf/crm_macro.xacro (robot description, xacro)
@@ -58,8 +58,8 @@
     </joint>
     <link name="right_ur3_nozzle"/>
-    <joint name="right_ur3_wrist_3-nozzle" type="fixed">
-      <parent link="right_ur3_wrist_3_link" />
+    <joint name="right_ur3_tool0-nozzle" type="fixed">
+      <parent link="right_ur3_tool0" />
       <child link="right_ur3_nozzle" />
-      <origin xyz="-0.002415 0.023405 0.1368" rpy="${pi} 0 0" />
+      <origin xyz="0.002 0.05 0.1368" rpy="${pi} 0 0" />
     </joint>
   </xacro:macro>
