Commit message: Update end effector color

File: crm_single_robot_cell/crm_description/urdf/ur_macro.xacro (robot description, xacro)
@@ -376,6 +376,6 @@
           </geometry>
           <origin rpy="${-pi/2} 0 0" xyz="-0.021844 0.003186 0"/>
-          <material name="yellow">
-            <color rgba="1 1 0 1"/>  <!-- RGBA values for yellow; R=1, G=1, B=0, A=1 (opaque) -->
+          <material name="custom_gray">
+            <color rgba="0.24705882352941178 0.34509803921568627 0.40784313725490196 1"/>
           </material>
         </visual>

Commit message: Fix robot end effector orientation

File: crm_single_robot_cell/crm_description/urdf/ur_macro.xacro (robot description, xacro)
@@ -375,5 +375,5 @@
             <mesh filename="package://crm_description/meshes/end_effector.stl"/>
           </geometry>
-          <origin rpy="${-pi/2} 0 0" xyz="-0.021844 0.003186 0"/>
+          <origin rpy="${-pi/2} 0 ${-pi/2}" xyz="0.003186 0.021844 0"/>
           <material name="custom_gray">
             <color rgba="0.24705882352941178 0.34509803921568627 0.40784313725490196 1"/>
@@ -384,5 +384,5 @@
             <mesh filename="package://crm_description/meshes/end_effector.stl"/>
           </geometry>
-          <origin rpy="${-pi/2} 0 0" xyz="-0.021844 0.003186 0"/>
+          <origin rpy="${-pi/2} 0 ${-pi/2}" xyz="0.003186 0.021844 0"/>
         </collision>
     </link>

Commit message: Update end effector stl for thermal camera mount

File: crm_single_robot_cell/crm_description/urdf/ur_macro.xacro (robot description, xacro)
@@ -306,5 +306,5 @@
         <visual>
           <geometry>
-            <mesh filename="package://crm_description/meshes/end_effector.stl"/>
+            <mesh filename="package://crm_description/meshes/end_effector_thermal_camera.stl"/>
           </geometry>
           <origin rpy="${-pi/2} 0 ${-pi/2}" xyz="0.003186 0.021844 0"/>
@@ -315,5 +315,5 @@
         <collision>
           <geometry>
-            <mesh filename="package://crm_description/meshes/end_effector.stl"/>
+            <mesh filename="package://crm_description/meshes/end_effector_thermal_camera.stl"/>
           </geometry>
           <origin rpy="${-pi/2} 0 ${-pi/2}" xyz="0.003186 0.021844 0"/>

Commit message: Fix displaying end effector

File: crm_single_robot_cell/crm_description/urdf/ur_macro.xacro (robot description, xacro)
@@ -304,5 +304,5 @@
     <!-- ROS-Industrial 'tool0' frame - all-zeros tool frame -->
     <link name="${tf_prefix}tool0">
-        <!-- <visual>
+        <visual>
           <geometry>
             <mesh filename="package://crm_description/meshes/end_effector_thermal_camera.stl"/>
@@ -318,5 +318,5 @@
           </geometry>
           <origin rpy="${-pi/2} 0 ${-pi/2}" xyz="0.003186 0.021844 0"/>
-        </collision> -->
+        </collision>
     </link>
     <joint name="${tf_prefix}flange-tool0" type="fixed">

Commit message: Tune servbo config

File: crm_single_robot_cell/crm_description/urdf/ur_macro.xacro (robot description, xacro)
@@ -322,5 +322,5 @@
     <joint name="${tf_prefix}flange-tool0" type="fixed">
       <!-- default toolframe - X+ left, Y+ up, Z+ front -->
-      <origin xyz="0 0 0" rpy="0 0 0"/>
+      <origin xyz="0 0 0" rpy="${pi/2.0} 0 ${pi/2.0}"/>
       <parent link="${tf_prefix}flange"/>
       <child link="${tf_prefix}tool0"/>
