Commit message: Set initial position

File: crm_dual_robot_cell/crm_dual_control/urdf/crm_dual_controlled.urdf.xacro (robot description, xacro)
@@ -35,4 +35,8 @@
   <xacro:arg name="ur_output_recipe_filename" default="$(find ur_robot_driver)/resources/rtde_output_recipe.txt" />
   <xacro:arg name="ur_input_recipe_filename" default="$(find ur_robot_driver)/resources/rtde_input_recipe.txt" />
+  <xacro:arg name="alice_initial_positions_file" default="$(find crm_dual_control)/config/alice_initial_positions.yaml"/>
+  <xacro:property name="alice_initial_positions_file" default="$(arg alice_initial_positions_file)"/>
+  <xacro:arg name="bob_initial_positions_file" default="$(find crm_dual_control)/config/bob_initial_positions.yaml"/>
+  <xacro:property name="bob_initial_positions_file" default="$(arg bob_initial_positions_file)"/>
   <link name="world" />
   <xacro:crm_dual_robot
@@ -66,4 +70,5 @@
     script_command_port="$(arg alice_script_command_port)"
     trajectory_port="$(arg alice_trajectory_port)"
+    initial_positions="${xacro.load_yaml(alice_initial_positions_file)}"
   />
   <xacro:ur_ros2_control
@@ -82,4 +87,5 @@
     script_command_port="$(arg bob_script_command_port)"
     trajectory_port="$(arg bob_trajectory_port)"
+    initial_positions="${xacro.load_yaml(bob_initial_positions_file)}"
   />
 </robot>

Commit message: Fix vention bench height in dual arm urdf

File: crm_dual_robot_cell/crm_dual_control/urdf/crm_dual_controlled.urdf.xacro (robot description, xacro)
@@ -53,5 +53,5 @@
     bob_visual_parameters_file="$(arg bob_visual_parameters_file)"
   >
-    <origin xyz="0 0 1" rpy="0 0 0" />
+    <origin xyz="0 0 0.776572" rpy="0 0 0" />
   </xacro:crm_dual_robot>
   <xacro:ur_ros2_control
