Commit message: Update driver launch for rolling

File: crm_single_robot_cell/crm_control/urdf/crm_controlled.urdf.xacro (robot description, xacro)
@@ -28,10 +28,10 @@
     visual_parameters_file="$(arg visual_parameters_file)"
   >
-    <origin xyz="0 0 0.78" rpy="0 0 0" />
+    <origin xyz="0 0 0.776572" rpy="0 0 0" />
   </xacro:crm_robot>
   <!--Create the control tag for the UR robot-->
   <xacro:ur_ros2_control
-    name="$(arg ur_type)"
-    tf_prefix="$(arg ur_type)_"
+    name="right_ur3"
+    tf_prefix="right_ur3_"
     kinematics_parameters_file="$(arg kinematics_parameters_file)"
     robot_ip="$(arg robot_ip)"

Commit message: Add initial_position to control launch

File: crm_single_robot_cell/crm_control/urdf/crm_controlled.urdf.xacro (robot description, xacro)
@@ -18,4 +18,6 @@
   <xacro:arg name="use_mock_hardware" default="false" />
   <xacro:arg name="mock_sensor_commands" default="false" />
+  <xacro:arg name="initial_positions_file" default="$(find crm_description)/config/initial_positions.yaml"/>
+  <xacro:property name="initial_positions_file" default="$(arg initial_positions_file)"/>
   <link name="world" />
   <!--Create the scene description including the robot-->
@@ -42,4 +44,5 @@
     mock_sensor_commands="$(arg mock_sensor_commands)"
     headless_mode="$(arg headless_mode)"
+    initial_positions="${xacro.load_yaml(initial_positions_file)}"
   />
   <!--If you had more controlled devices in your description, e.g. a gripper, you can add another ros2_control tag here-->

Commit message: Remove prefix

File: crm_single_robot_cell/crm_control/urdf/crm_controlled.urdf.xacro (robot description, xacro)
@@ -34,6 +34,6 @@
   <!--Create the control tag for the UR robot-->
   <xacro:ur_ros2_control
-    name="right_ur3"
-    tf_prefix="right_ur3_"
+    name="crm"
+    tf_prefix=""
     kinematics_parameters_file="$(arg kinematics_parameters_file)"
     robot_ip="$(arg robot_ip)"

File: crm_single_robot_cell/crm_description/urdf/crm_macro.xacro (robot description, xacro)
@@ -41,6 +41,6 @@
     <!--This will create the specific robot-->
     <xacro:ur_robot
-      name="right_ur3"
-      tf_prefix="right_ur3_"
+      name="crm"
+      tf_prefix=""
       parent="robot_mount"
       joint_limits_parameters_file="${joint_limits_parameters_file}"
@@ -51,14 +51,14 @@
       <origin xyz="0 0 0" rpy="0 0 0" />
     </xacro:ur_robot>
-    <link name="right_ur3_bltouch"/>
-    <joint name="right_ur3_wrist_3-bltouch" type="fixed">
-      <parent link="right_ur3_wrist_3_link" />
-      <child link="right_ur3_bltouch" />
+    <link name="bltouch"/>
+    <joint name="wrist_3-bltouch" type="fixed">
+      <parent link="wrist_3_link" />
+      <child link="bltouch" />
       <origin xyz="0.0674 0 0.0206502" rpy="0 ${pi/2} ${pi}" />
     </joint>
-    <link name="right_ur3_nozzle"/>
-    <joint name="right_ur3_tool0-nozzle" type="fixed">
-      <parent link="right_ur3_tool0" />
-      <child link="right_ur3_nozzle" />
+    <link name="nozzle"/>
+    <joint name="tool0-nozzle" type="fixed">
+      <parent link="tool0" />
+      <child link="nozzle" />
       <origin xyz="0.002 0.05 0.1368" rpy="${pi} 0 0" />
     </joint>
